File: KiCad/Green Pill/Green Pill.kicad_pcb (KiCad board)
At the start: 2 copper layers, 51.2 x 70.4 mm, 29 parts, among them J1 10103594-0001LF, J2 68000-220HLF, J3 0022232041, J4 M20-9980345, J5 68000-220HLF, U1 STM32F103C8Tx, U2 AZ1117-3.3, Y1 8MHz, Y2 32.768kHz

Commit message: corrigi o projeto
Parts:
- added REF**: OSHW-Logo2_7.3x6mm_SilkScreen, Symbol:OSHW-Logo2_7.3x6mm_SilkScreen, F.Cu at (131.6, 121.4)
Routing:
- net Net-(J5-Pad14): track 20.5 -> 22.2 mm
- net Net-(J5-Pad16): track 24.2 -> 25.8 mm
- net Net-(J5-Pad15): track 22.3 -> 23.5 mm
- net PB12: track 32.1 -> 33.2 mm
- net PB15: track 26.3 -> 27.3 mm
- net PC14-OSC_IN: track 53.3 -> 52.3 mm
- net PB13: track 30.2 -> 31.2 mm
- net PB14: track 28.2 -> 29.3 mm
- net RESET: track 85.3 -> 86.0 mm
- net PA11-USART_CTS: track 19.5 -> 20.2 mm
- net Net-(J2-Pad16): track 33.7 -> 34.3 mm
- net PB7: track 24.6 -> 24.8 mm, vias 0 -> 1
- net PB9: vias 0 -> 1
- net PB8: vias 0 -> 1
- net PB6: vias 0 -> 1
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Other:
- board text added: "+3.3V"
- board text added: "CLK"
- board text added: "GND"
- board text added: "ILS (Green Pill v.20200404)"
- board text added: "IO"
- board text added: "KiCad 5.1.4"

Commit message: corrigi o projeto
Other:
- board text added: "BT0"
- board text added: "BT1"
Changed lines of the file:
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@@
   (general
     (thickness 1.6)
-    (drawings 10)
+    (drawings 14)
     (tracks 729)
     (zones 0)
@@
   )
   (setup
-    (last_trace_width 0.25)
+    (last_trace_width 1.25)
     (user_trace_width 0.25)
     (user_trace_width 0.5)
@@
     (descr "Through hole straight pin header, 2x03, 2.54mm pitch, double rows")
     (tags "Through hole pin header THT 2x03 2.54mm double row")
-    (fp_text reference J4 (at 3.82 -2.91 180) (layer F.SilkS)
+    (fp_text reference J4 (at 4.28 -2.72 180) (layer F.SilkS)
       (effects (font (size 1 1) (thickness 0.15)))
     )
@@
     )
   )
+  (gr_text +3.3V (at 162.8 76.97 90) (layer F.SilkS)
+    (effects (font (size 0.75 0.75) (thickness 0.15)))
+  )
+  (gr_text GND (at 157.63 67.65 90) (layer F.SilkS)
+    (effects (font (size 0.75 0.75) (thickness 0.15)))
+  )
+  (gr_text BT1 (at 165.66 70.84) (layer F.SilkS)
+    (effects (font (size 0.75 0.75) (thickness 0.15)))
+  )
+  (gr_text BT0 (at 165.66 73.33) (layer F.SilkS)
+    (effects (font (size 0.75 0.75) (thickness 0.15)))
+  )
   (gr_text CLK (at 152.82 65.3 90) (layer F.SilkS)

Commit message: corrigi o projeto
Parts:
- renumbered B3F-1000 to RESET
Other:
- board text added: "+3V3"
- board text added: "+5V"
- board text added: "PA0-WKUP"
- board text added: "PA1"
- board text added: "PA10"
- board text added: "PA11"
- board text added: "PA12"
- board text added: "PA15"
- board text added: "PA2"
- board text added: "PA3"
- board text added: "PA4"
- board text added: "PA5"
- board text added: "PA6"
- board text added: "PA7"
- board text added: "PA8"
- board text added: "PA9"
- board text added: "PB0"
- board text added: "PB1"
- board text added: "PB10"
- board text added: "PB11"
- board text added: "PB12"
- board text added: "PB13"
- board text added: "PB14"
- board text added: "PB15"
- board text added: "PB3"
- board text added: "PB4"
- board text added: "PB5"
- board text added: "PB6"
- board text added: "PB7"
- board text added: "PB8"
- board text added: "PB9"
- board text added: "PC13"
- board text added: "PC14-OSC_IN"
- board text added: "PC15-OSC_OUT"
- board text added: "RESET"
- board text added: "VBAT"
