File: KiCad/Green Pill/Green Pill.sch (KiCad schematic (older format))
At the start: 29 parts, among them J1 10103594-0001LF, J2 68000-220HLF, J3 0022232041, J4 M20-9980345, J5 68000-220HLF, U1 STM32F103C8Tx, U2 AZ1117-3.3, Y1 8MHz, Y2 32.768kHz

Commit message: corrigi o projeto
Parts:
- R3: value 10k -> 1.5k
Changed lines of the file:
@@
 EESchema Schematic File Version 4
+LIBS:Green Pill-cache
 EELAYER 30 0
 EELAYER END
@@
 P 3950 4600
 F 0 "R3" H 3880 4554 50  0000 R CNN
-F 1 "10k" H 3880 4645 50  0000 R CNN
+F 1 "1.5k" H 3880 4645 50  0000 R CNN
 F 2 "Resistor_THT:R_Axial_DIN0207_L6.3mm_D2.5mm_P7.62mm_Horizontal" V 3880 4600 50  0001 C CNN
 F 3 "~" H 3950 4600 50  0001 C CNN
